Commit message: Add files via upload

File: my_robot/my_robot_gazebo/urdf/my_robot.gazebo.xacro (robot description, xacro)
@@ -3,26 +3,4 @@
 	<xacro:include filename="$(find my_robot_description)/urdf/00-agricole.xacro" />
 	<gazebo>
-		<!--
-		<plugin name="differential_drive_controller" filename="libgazebo_ros_diff_drive.so">
-        		<alwaysOn>true</alwaysOn>
-        		<updateRate>40</updateRate>
-        		<legacyMode>false</legacyMode>
-        		<leftJoint>rr_wheel_joint</leftJoint>
-        		<rightJoint>rl_wheel_joint</rightJoint>
-        		<wheelSeparation>0.39</wheelSeparation>
-        		<wheelDiameter>0.15</wheelDiameter>
-        		<torque>5</torque>
-        		<commandTopic>cmd_vel</commandTopic>
-        		<odometryTopic>odom</odometryTopic>
-        		<odometryFrame>odom</odometryFrame>
-        		<robotBaseFrame>base_link</robotBaseFrame>
-        		<publishWheelTF>false</publishWheelTF>
-        		<publishWheelJointState>false</publishWheelJointState>
-        		<rosDebugLevel>na</rosDebugLevel>
-        		<wheelAcceleration>0</wheelAcceleration>
-        		<wheelTorque>5</wheelTorque>
-        		<odometrySource>world</odometrySource>
-        		<publishTf>1</publishTf>
-    		</plugin> -->
 		<plugin name="gazebo_ros_control" filename="libgazebo_ros_control.so">
 			<robotNamespace>/</robotNamespace>
@@ -50,3 +28,6 @@
 	<xacro:wheel_trans_macro pos="rl"/>
 	<xacro:wheel_trans_macro pos="rr"/>
+		<!--gazebo reference="base_link">
+			<material>Gazebo/Blue</material>
+		</gazebo-->
 </robot>

Commit message: Add files via upload

File: my_robot/my_robot_gazebo/urdf/my_robot.gazebo.xacro (robot description, xacro)
@@ -1,5 +1,7 @@
 <?xml version="1.0"?>
 <robot xmlns:xacro="http://www.ros.org/wiki/xacro" name="my_robot">
-	<xacro:include filename="$(find my_robot_description)/urdf/00-agricole.xacro" />
+    <!--Fichier d'appel du xacro du robot agricole-->
+	<xacro:include filename="$(find my_robot_description)/urdf/01-agricole.xacro" />
+<!--Implementation des plugins necessaires-->
 	<gazebo>
 		<plugin name="gazebo_ros_control" filename="libgazebo_ros_control.so">
@@ -8,4 +10,100 @@
 		</plugin>
 	</gazebo>
+	<!--Plugins de la camera-->
+	<gazebo reference="camera">
+    		<material>Gazebo/Green</material>
+    		<sensor type="camera" name="camera">
+      			<update_rate>30.0</update_rate>
+      			<camera name="head">
+        			<horizontal_fov>1.3962634</horizontal_fov>
+        			<image>
+          				<width>800</width>
+          				<height>800</height>
+          				<format>R8G8B8</format>
+        			</image>
+        			<clip>
+          				<near>0.02</near>
+          				<far>300</far>
+        			</clip>
+      			</camera>
+      			<plugin name="camera_controller" filename="libgazebo_ros_camera.so">
+        			<alwaysOn>true</alwaysOn>
+        			<updateRate>0.0</updateRate>
+        			<cameraName>mybot/camera</cameraName>
+        			<imageTopicName>image_raw</imageTopicName>
+        			<cameraInfoTopicName>camera_info</cameraInfoTopicName>
+       				<frameName>camera</frameName>
+        			<hackBaseline>0.07</hackBaseline>
+        			<distortionK1>0.0</distortionK1>
+        			<distortionK2>0.0</distortionK2>
+        			<distortionK3>0.0</distortionK3>
+        			<distortionT1>0.0</distortionT1>
+        			<distortionT2>0.0</distortionT2>
+      			</plugin>
+    		</sensor>
+  	</gazebo>
+	<!--Plugins de l'imu-->
+	<gazebo reference="imu">
+    		<material>Gazebo/Black</material>
+		<sensor name="imu" type="imu">
+        		<imu>
+          			<angular_velocity>
+            				<x>
+              					<noise type="gaussian">
+                					<mean>0.0</mean>
+                					<stddev>2e-4</stddev>
+                					<bias_mean>0.0000075</bias_mean>
+                					<bias_stddev>0.0000008</bias_stddev>
+              					</noise>
+           				 </x>
+           				 <y>
+              					<noise type="gaussian">
+                					<mean>0.0</mean>
+                					<stddev>2e-4</stddev>
+                					<bias_mean>0.0000075</bias_mean>
+                					<bias_stddev>0.0000008</bias_stddev>
+             					</noise>
+           				</y>
+            				<z>
+             					<noise type="gaussian">
+                					<mean>0.0</mean>
+                					<stddev>2e-4</stddev>
+                					<bias_mean>0.0000075</bias_mean>
+                					<bias_stddev>0.0000008</bias_stddev>
+             					</noise>
+            				</z>
+          			</angular_velocity>
+          			<linear_acceleration>
+            				<x>
+              					<noise type="gaussian">
+                					<mean>0.0</mean>
+                					<stddev>1.7e-2</stddev>
+                					<bias_mean>0.1</bias_mean>
+                					<bias_stddev>0.001</bias_stddev>
+              					</noise>
+            				</x>
+           				<y>
+              					<noise type="gaussian">
+                					<mean>0.0</mean>
+                					<stddev>1.7e-2</stddev>
+                					<bias_mean>0.1</bias_mean>
+                					<bias_stddev>0.001</bias_stddev>
+              					</noise>
+            				</y>
+            				<z>
+              					<noise type="gaussian">
+                					<mean>0.0</mean>
+                					<stddev>1.7e-2</stddev>
+                					<bias_mean>0.1</bias_mean>
+                					<bias_stddev>0.001</bias_stddev>
+              					</noise>
+            				</z>
+          			</linear_acceleration>
+        		</imu>
+        		<always_on>1</always_on>
+        		<update_rate>1000</update_rate>
+      		</sensor>
+	</gazebo>
+	<!--Plugins des roues motrices-->
 	<xacro:macro name="wheel_trans_macro" params="pos">
 		<transmission name = "${pos}_wheel_trans">
@@ -26,8 +124,6 @@
 		</gazebo>
 	</xacro:macro>
+	<!--Appel de nos deux roues motrices (roues arrieres)-->
 	<xacro:wheel_trans_macro pos="rl"/>
 	<xacro:wheel_trans_macro pos="rr"/>
-		<!--gazebo reference="base_link">
-			<material>Gazebo/Blue</material>
-		</gazebo-->
 </robot>
