Commit message: Add files via upload

File: my_robot/my_robot_description/urdf/01-agricole.xacro (robot description, xacro)
@@ -172,3 +172,23 @@
       <child link="imu"/>
     </joint>
+  <!-- Hokuyo Laser -->
+    <joint name="hokuyo_joint" type="fixed">
+    <axis xyz="0 1 0" />
+    <origin xyz="-0.15 0 0.15" rpy="0 0 0"/>
+    <parent link="base_link"/>
+    <child link="hokuyo"/>
+  </joint>
+  <link name="hokuyo">
+    <visual>
+      <origin xyz="0 0 0" rpy="0 0 0"/>
+      <geometry>
+        <mesh filename="package://my_robot_description/meshes/hokuyo.dae"/>
+      </geometry>
+    </visual>
+    <inertial>
+      <mass value="1e-5" />
+      <origin xyz="0 0 0" rpy="0 0 0"/>
+      <inertia ixx="1e-6" ixy="0" ixz="0" iyy="1e-6" iyz="0" izz="1e-6" />
+    </inertial>
+  </link>
 </robot>

File: my_robot/my_robot_gazebo/urdf/my_robot.gazebo.xacro (robot description, xacro)
@@ -105,4 +105,37 @@
       		</sensor>
 	</gazebo>
+	<!-- hokuyo -->
+  	<gazebo reference="hokuyo">
+    		<sensor type="gpu_ray" name="head_hokuyo_sensor">
+      			<pose>0 0 0 0 0 0</pose>
+			<!-- visualize sert a visualiser ou non la detection d'obstacles sur Gazebo ainsi si on met true alors on affichera le faisceau du lidar sur gazebo -->
+      			<visualize>true</visualize>
+      			<update_rate>40</update_rate>
+      			<ray>
+        			<scan>
+          				<horizontal>
+            					<samples>720</samples>
+            					<resolution>1</resolution>
+            					<min_angle>-1.570796</min_angle>
+            					<max_angle>1.570796</max_angle>
+          				</horizontal>
+        			</scan>
+        			<range>
+          				<min>0.10</min>
+          				<max>30.0</max>
+          				<resolution>0.01</resolution>
+        			</range>
+        			<noise>
+          				<type>gaussian</type>
+          				<mean>0.0</mean>
+          				<stddev>0.01</stddev>
+        			</noise>
+      			</ray>
+      			<plugin name="gazebo_ros_head_hokuyo_controller" filename="libgazebo_ros_gpu_laser.so">
+        			<topicName>/mybot/laser/scan</topicName>
+        			<frameName>hokuyo</frameName>
+      			</plugin>
+    		</sensor>
+  	</gazebo>
 	<!--Plugins des roues motrices-->
 	<xacro:macro name="wheel_trans_macro" params="pos">
